File: bike-alarm.sch (EAGLE design)
At the start: 31 parts, among them Q1 8.00M-SMDHC, U1 MCP73833, U6 ATMEGA32U4-AU

Commit message: More stuff
Parts:
- added C10, C11: 1uF, microbuilder:CAP_CERAMIC0603
- added U$1: MCP1700, my:MCP1700
Connections:
- new net 3V: C11.P$1, U$1.VOUT
- net GND: now also C10.P$2, C11.P$2, U$1.GND
- net VBAT: now also C10.P$1, U$1.VIN
Other:
- note added: "3V regulator"
Changed lines of the file:
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@@
 <setting verticaltext="up"/>
 </settings>
-<grid distance="0.1" unitdist="inch" unit="inch" style="lines" multiple="1" display="no" altdistance="0.01" altunitdist="inch" altunit="inch"/>
+<grid distance="0.05" unitdist="inch" unit="inch" style="lines" multiple="1" display="no" altdistance="0.01" altunitdist="inch" altunit="inch"/>
 <layers>
 <layer number="1" name="Top" color="4" fill="1" visible="no" active="no"/>
@@
 <layer number="112" name="tSilk" color="7" fill="1" visible="no" active="yes"/>
 <layer number="113" name="ReferenceLS" color="7" fill="1" visible="no" active="no"/>
+<layer number="114" name="Badge_Outline" color="7" fill="1" visible="yes" active="yes"/>
+<layer number="115" name="ReferenceISLANDS" color="7" fill="1" visible="yes" active="yes"/>
 <layer number="116" name="Patch_BOT" color="9" fill="4" visible="no" active="yes"/>
 <layer number="118" name="Rect_Pads" color="7" fill="1" visible="no" active="no"/>
@@
 <part name="R3" library="microbuilder" deviceset="RESISTOR" device="_0603" value="22"/>
 <part name="VBUS" library="my" deviceset="VBUS" device=""/>
-<part name="U$2" library="my" deviceset="VBAT" device=""/>
-<part name="U$3" library="my" deviceset="VBAT" device=""/>
+<part name="U$2" library="my" deviceset="3V" device=""/>
+<part name="U$3" library="my" deviceset="3V" device=""/>
 <part name="U1" library="microbuilder" deviceset="MCP73833" device="" value="MCP73833"/>
 <part name="LED1" library="adafruit" deviceset="LED" device="3MM" value="ORANGE"/>
@@
 <part name="GND6" library="supply1" deviceset="GND" device=""/>
 <part name="U$4" library="my" deviceset="TPS61085" device=""/>
-<part name="U$5" library="my" deviceset="VBAT" device=""/>
+<part name="U$5" library="my" deviceset="3V" device=""/>
 <part name="C3" library="microbuilder" deviceset="CAP_CERAMIC" device="0603" value="1uF"/>
 <part name="C4" library="microbuilder" deviceset="CAP_CERAMIC" device="0805" value="10uF 16V"/>
@@
 <part name="C9" library="microbuilder" deviceset="CAP_CERAMIC" device="0603" value="1uF"/>
 <part name="GND8" library="supply1" deviceset="GND" device=""/>
-<part name="U$8" library="my" deviceset="VBAT" device=""/>
+<part name="U$8" library="my" deviceset="3V" device=""/>
+<part name="U$1" library="my" deviceset="MCP1700" device=""/>
+<part name="U$6" library="my" deviceset="VBAT" device=""/>
+<part name="U$9" library="my" deviceset="3V" device=""/>
+<part name="GND10" library="supply1" deviceset="GND" device=""/>
+<part name="C10" library="microbuilder" deviceset="CAP_CERAMIC" device="0603" value="1uF"/>
+<part name="C11" library="microbuilder" deviceset="CAP_CERAMIC" device="0603" value="1uF"/>
 </parts>
 <sheets>
 <sheet>
 <plain>
-<text x="91.44" y="248.92" size="1.778" layer="94">MicroUSB connection</text>
-<text x="104.14" y="149.86" size="1.778" layer="94">Battery charger</text>
-<text x="218.44" y="147.32" size="1.778" layer="94">DC-DC Converter 12V</text>
+<text x="91.44" y="248.92" size="1.778" layer="97">MicroUSB connection</text>
+<text x="104.14" y="149.86" size="1.778" layer="97">Battery charger</text>
+<text x="218.44" y="147.32" size="1.778" layer="97">DC-DC Converter 12V</text>
+<text x="96.52" y="201.93" size="1.778" layer="97">3V regulator</text>
 </plain>
 <instances>
@@
 <instance part="R3" gate="G$1" x="110.49" y="232.41"/>
 <instance part="VBUS" gate="VBUS" x="102.87" y="236.22"/>
-<instance part="U$2" gate="VBAT" x="129.54" y="130.81"/>
-<instance part="U$3" gate="VBAT" x="160.02" y="226.06"/>
+<instance part="U$2" gate="3V" x="129.54" y="130.81"/>
+<instance part="U$3" gate="3V" x="160.02" y="226.06"/>
 <instance part="U1" gate="G$1" x="111.76" y="119.38"/>
 <instance part="LED1" gate="G$1" x="86.36" y="142.24"/>
@@
 <instance part="GND6" gate="1" x="153.67" y="189.23" rot="R270"/>
 <instance part="U$4" gate="A" x="214.63" y="123.19"/>
-<instance part="U$5" gate="VBAT" x="185.42" y="132.08"/>
+<instance part="U$5" gate="3V" x="185.42" y="132.08"/>
 <instance part="C3" gate="G$1" x="191.77" y="119.38"/>
 <instance part="C4" gate="G$1" x="187.96" y="121.92" rot="R180"/>
@@
 <instance part="C9" gate="G$1" x="157.48" y="203.2" rot="R90"/>
 <instance part="GND8" gate="1" x="147.32" y="203.2" rot="R270"/>
-<instance part="U$8" gate="VBAT" x="229.87" y="220.98"/>
+<instance part="U$8" gate="3V" x="229.87" y="220.98"/>
+<instance part="U$1" gate="A" x="106.68" y="187.96"/>
+<instance part="U$6" gate="VBAT" x="86.36" y="196.85"/>
+<instance part="U$9" gate="3V" x="124.46" y="195.58"/>
+<instance part="GND10" gate="1" x="106.68" y="175.26"/>
+<instance part="C10" gate="G$1" x="90.17" y="185.42"/>
+<instance part="C11" gate="G$1" x="120.65" y="185.42"/>
 </instances>
 <busses>
@@
 <pinref part="GND8" gate="1" pin="GND"/>
 </segment>
+<segment>
+<pinref part="U$1" gate="A" pin="GND"/>
+<wire x1="106.68" y1="180.34" x2="106.68" y2="179.07" width="0.1524" layer="91"/>
+<pinref part="GND10" gate="1" pin="GND"/>
+<pinref part="C10" gate="G$1" pin="P$2"/>
+<wire x1="106.68" y1="179.07" x2="106.68" y2="177.8" width="0.1524" layer="91"/>
+<wire x1="90.17" y1="182.88" x2="90.17" y2="179.07" width="0.1524" layer="91"/>
+<wire x1="90.17" y1="179.07" x2="106.68" y2="179.07" width="0.1524" layer="91"/>
+<wire x1="106.68" y1="179.07" x2="120.65" y2="179.07" width="0.1524" layer="91"/>
+<pinref part="C11" gate="G$1" pin="P$2"/>
+<wire x1="120.65" y1="179.07" x2="120.65" y2="182.88" width="0.1524" layer="91"/>
+<junction x="106.68" y="179.07"/>
+</segment>
 </net>
 <net name="N$1" class="0">
@@
 <net name="VBAT" class="0">
 <segment>
-<pinref part="U$2" gate="VBAT" pin="VBAT"/>
+<pinref part="U$2" gate="3V" pin="3V"/>
 <wire x1="129.54" y1="127" x2="129.54" y2="130.81" width="0.1524" layer="91"/>
 <pinref part="U1" gate="G$1" pin="VBAT1"/>
@@
 </segment>
 <segment>
-<pinref part="U$3" gate="VBAT" pin="VBAT"/>
+<pinref part="U$3" gate="3V" pin="3V"/>
 <wire x1="160.02" y1="226.06" x2="160.02" y2="223.52" width="0.1524" layer="91"/>
 <pinref part="U6" gate="G$1" pin="AVCC1"/>
@@
 </segment>
 <segment>
-<pinref part="U$5" gate="VBAT" pin="VBAT"/>
+<pinref part="U$5" gate="3V" pin="3V"/>
 <wire x1="185.42" y1="127" x2="185.42" y2="132.08" width="0.1524" layer="91"/>
 <pinref part="C4" gate="G$1" pin="P$2"/>
@@
 <pinref part="U6" gate="G$1" pin="PE2(!HWB)"/>
 <wire x1="218.44" y1="220.98" x2="229.87" y2="220.98" width="0.1524" layer="91"/>
-<pinref part="U$8" gate="VBAT" pin="VBAT"/>
+<pinref part="U$8" gate="3V" pin="3V"/>
+</segment>
+<segment>
+<pinref part="U$1" gate="A" pin="VIN"/>
+<wire x1="96.52" y1="193.04" x2="90.17" y2="193.04" width="0.1524" layer="91"/>
+<wire x1="90.17" y1="193.04" x2="86.36" y2="193.04" width="0.1524" layer="91"/>
+<wire x1="86.36" y1="193.04" x2="86.36" y2="196.85" width="0.1524" layer="91"/>
+<pinref part="U$6" gate="VBAT" pin="VBAT"/>
+<pinref part="C10" gate="G$1" pin="P$1"/>
+<wire x1="90.17" y1="190.5" x2="90.17" y2="193.04" width="0.1524" layer="91"/>
+<junction x="90.17" y="193.04"/>
 </segment>
 </net>
@@
 </segment>
 </net>
+<net name="3V" class="0">
+<segment>
+<pinref part="U$1" gate="A" pin="VOUT"/>
+<wire x1="116.84" y1="193.04" x2="120.65" y2="193.04" width="0.1524" layer="91"/>
+<wire x1="120.65" y1="193.04" x2="124.46" y2="193.04" width="0.1524" layer="91"/>
+<wire x1="124.46" y1="193.04" x2="124.46" y2="195.58" width="0.1524" layer="91"/>
+<pinref part="U$9" gate="3V" pin="3V"/>
+<pinref part="C11" gate="G$1" pin="P$1"/>
+<wire x1="120.65" y1="190.5" x2="120.65" y2="193.04" width="0.1524" layer="91"/>
+<junction x="120.65" y="193.04"/>
+</segment>
+</net>
